File: SX1255-SXCEIVER-HAT.kicad_pcb (KiCad board)
At the start: 2 copper layers, 65 x 56.2 mm, 84 parts, among them IC1 SX1255, J1 U.FL, J2 U.FL, J3 RPi, J4 WP, Q1 BSS84, U1 MCP1703Ax-330xxDB, U2 24LC256, U3 74LVC1G74DP_125, U4 TQP3M9036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

Commit message: Add files via upload
Other:
- board text added: "V1.3"
- board text added: "Z32IT"
Changed lines of the file:
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@@
 		(tags "resistor")
 		(property "Reference" "R3"
-			(at -4 0 90)
+			(at 0 1.5 90)
 			(layer "F.SilkS")
 			(effects
@@
 		(layer "Edge.Cuts")
 	)
+	(gr_text "V1.3"
+		(at 135.75 118.75 0)
+		(layer "F.SilkS")
+		(effects
+			(font
+				(size 1.5 1.5)
+				(thickness 0.3)
+				(bold yes)
+			)
+			(justify left bottom)
+		)
+	)
 	(gr_text "RX"
 		(at 114 124 0)
@@
 				(bold yes)
 			)
+			(justify left bottom)
+		)
+	)
+	(gr_text "Z32IT"
+		(at 121 119 0)
+		(layer "F.SilkS")
+		(effects
+			(font
+				(size 1.5 1.5)
+				(thickness 0.3)
+				(bold yes)
+			)

Commit message: Add files via upload
Parts:
- moved FL1 2.00 mm to (153.2, 112.2)
- moved J2 2.00 mm to (153.2, 120.3)
- moved R27 2.00 mm to (154.0, 116.8)
Routing:
- net Net-(FL1-IN): track 2.78 -> 4.78 mm
- net GND: vias 144 -> 68

Commit message: Add files via upload
Parts:
- moved J2 11.9 mm to (160.4, 110.8), turned to 180 degrees
- moved J1 11.1 mm to (109.2, 110.8), turned to 0 degrees
- moved R27 5.81 mm to (156.9, 111.8), turned to 90 degrees
- moved R26 5.15 mm to (113.0, 111.8), turned to 90 degrees
- moved FL1 1.51 mm to (153.4, 110.8), turned to 0 degrees
- moved REF** 0.25 mm to (132.0, 118.8)
Routing:
- net Net-(FL2-IN): track 8.12 -> 4.38 mm
- net Net-(FL1-IN): track 4.78 -> 3.30 mm
- net Net-(FL1-OUT): track 4.88 -> 3.85 mm
- net GND: vias 68 -> 37
Other:
- board text added: "DIO0"
- board text added: "DIO1"
- board text added: "DIO3"
- board text added: "PA"
- board text added: "POW"
- board text added: "m/SXceiver"

Commit message: Add files via upload
Parts:
- removed F1: 6V/0.5A, Fuse:Fuse_1206_3216Metric
- added D2: Green, LED_SMD:LED_0603_1608Metric_Pad1.05x0.95mm_HandSolder, F.Cu at (158.2, 91.0)
- added D3: Red, LED_SMD:LED_0603_1608Metric_Pad1.05x0.95mm_HandSolder, F.Cu at (160.0, 91.0)
- added R34: 1K, Resistor_SMD:R_0603_1608Metric, F.Cu at (158.2, 87.5)
- added R35: 330R, Resistor_SMD:R_0603_1608Metric, F.Cu at (160.0, 87.5)
- L4: footprint Capacitor_SMD:C_0603_1608Metric -> Inductor_SMD:L_0603_1608Metric
- Y1: value TCXO 38.40MHz -> 38.4MHz; footprint Crystal:Crystal_SMD_3225-4Pin_3.2x2.5mm -> Oscillator:Oscillator_SMD_ECS_2520MV-xxx-xx-4Pin_2.5x2.0mm
- moved C1 7.16 mm to (110.0, 79.2), turned to 0 degrees
- moved L1 2.14 mm to (106.8, 80.0)
- moved Y1 0.26 mm to (146.8, 96.0), turned to -90 degrees
Connections:
- C1 pad 1: Net-(C1-Pad1) -> +5VP
- L1 pad 1: Net-(C1-Pad1) -> +5VP
- U4 pad 1: GND -> (no net)
- U4 pad 3: GND -> (no net)
- U4 pad 4: GND -> (no net)
- U4 pad 5: GND -> (no net)
- U4 pad 8: GND -> (no net)
Routing:
- net /H_GPIO12: track 0.00 -> 25.8 mm, vias 0 -> 2
- net /H_GPIO13: track 0.00 -> 21.2 mm, vias 0 -> 2
- net +5VP: track 10.4 -> 14.6 mm
- net Net-(C1-Pad1): track 3.87 -> 0.00 mm
- net Net-(D3-A): track 0.00 -> 1.80 mm
- net Net-(D2-A): track 0.00 -> 1.80 mm
- net /H_CE0: track 58.3 -> 59.2 mm
- net +5V: track 97.2 -> 98.0 mm
- net GND: vias 37 -> 33
Other:
- board text added: "GPIO12"
- board text added: "GPIO13"
- board text added: "V1.3.1"
- board text removed: "V1.3"
