File: SX1255-SXCEIVER-HAT.kicad_pcb (KiCad board)
At the start: 2 copper layers, 65 x 56.2 mm, 87 parts, among them IC1 SX1255, J1 U.FL, J2 U.FL, J3 RPi, J4 WP, Q1 BSS84, U1 MCP1703Ax-330xxDB, U2 24LC256, U3 74LVC1G74DP_125, U4 TQP3M9036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

Commit message: Add files via upload
Parts:
- added JP1: With/Without U3, Jumper:SolderJumper-2_P1.3mm_Open_RoundedPad1.0x1.5mm, F.Cu at (150.8, 99.8)
- L1: footprint Inductor_SMD:L_0603_1608Metric -> Inductor_SMD:L_0805_2012Metric
- Y1: value 38.4MHz -> 38.4MHZ; footprint Oscillator:Oscillator_SMD_ECS_2520MV-xxx-xx-4Pin_2.5x2.0mm -> Crystal:Crystal_SMD_3225-4Pin_3.2x2.5mm
- moved C28 2.09 mm to (149.4, 112.0)
- moved FL2 1.95 mm to (118.2, 111.9)
- moved C30 1.77 mm to (146.0, 117.5)
- moved C31 1.77 mm to (146.0, 115.8)
- moved L4 1.77 mm to (146.8, 112.8)
- moved C17 1.50 mm to (132.8, 112.0)
- moved FL1 1.32 mm to (153.9, 112.0)
- moved J2 1.32 mm to (160.9, 112.0)
- moved R27 1.32 mm to (157.4, 113.0)
- moved C19 1.27 mm to (139.0, 112.0)
- moved J1 1.25 mm to (109.2, 112.0)
- moved L2 1.25 mm to (126.5, 114.5)
- moved L3 1.25 mm to (125.5, 112.0)
- moved U4 1.14 mm to (143.5, 112.2)
- moved R26 1.12 mm to (113.5, 112.8)
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Connections:
- U4 pad 1: (no net) -> GND
- U4 pad 3: (no net) -> GND
- U4 pad 4: (no net) -> GND
- U4 pad 5: (no net) -> GND
- U4 pad 8: (no net) -> GND
Routing:
- net /SX_VBAT3: track 17.1 -> 22.0 mm
- net Net-(JP1-A): track 3.76 -> 8.28 mm
- net +5V: track 98.0 -> 99.9 mm
- net Net-(FL2-IN): track 4.38 -> 5.88 mm
- net /SX_RFO_N: track 4.28 -> 5.78 mm
- net Net-(FL1-IN): track 3.30 -> 2.05 mm
- net /SX_RFI: track 9.85 -> 11.1 mm
- net Net-(FL2-OUT): track 6.09 -> 4.97 mm
- net /RF-out: track 5.27 -> 4.16 mm
- net +5VP: track 14.6 -> 13.8 mm
- net /SX_RFO_P: track 8.05 -> 8.80 mm
- net GND: vias 33 -> 280
Other:
- outline, holes or cut-outs redrawn
- board text added: "Final"
- board text added: "V1.3.2"
- board text removed: "V1.3.1"

Commit message: Add files via upload
Parts:
- Y1: value 38.4MHZ -> 38.4MHz
Connections:
- U4 pad 1: GND -> (no net)
- U4 pad 3: GND -> (no net)
- U4 pad 4: GND -> (no net)
- U4 pad 5: GND -> (no net)
- U4 pad 8: GND -> (no net)
Changed lines of the file:
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@@
 		(sheetname "/")
 		(sheetfile "SX1255-SXCEIVER-HAT.kicad_sch")
-		(attr smd)
+		(attr smd exclude_from_bom dnp)
 		(fp_line
 			(start -0.237258 -0.5225)
@@
 			)
 		)
-		(property "Description" "Inductor with ferrite core, small symbol"
+		(property "Description" "FERRITE BEAD 600 OHM 0805 1LN"
 			(at 0 0 270)
 			(unlocked yes)
@@
 			)
 		)
-		(property "Manufacturer Product Number" "BLM18HG601SN1D"
+		(property "Manufacturer Product Number" "BLM21BD601SN1D"
 			(at 0 0 270)
 			(unlocked yes)
@@
 			)
 		)
-		(property "Part Number" "490-1033-1-ND"
+		(property "Part Number" "490-1046-1-ND"
 			(at 0 0 270)
 			(unlocked yes)
@@
 			)
 		)
-		(property "Value" "38.4MHZ"
+		(property "Value" "38.4MHz"
 			(at 0 2.45 0)
 			(layer "F.Fab")
@@
 			)
 		)
-		(property "Description" "Clipped SW 0.5~1ppm"
+		(property "Description" "Clipped SW/0.5~1ppm"
 			(at 0 0 180)
 			(unlocked yes)
@@
 			)
 		)
+		(property "Manufacturer" "EPSON "
+			(at 0 0 180)
+			(unlocked yes)
+			(layer "F.Fab")
+			(hide yes)
+			(effects
+				(font
+					(size 1 1)
+					(thickness 0.15)
+				)
+			)
+		)
+		(property "Manufacturer Product Number" "TG2520SMN 38.4000M-MCGNNM3"
+			(at 0 0 180)
+			(unlocked yes)
+			(layer "F.Fab")
+			(hide yes)
+			(effects
+				(font
+					(size 1 1)
+					(thickness 0.15)
+				)
+			)
+		)
+		(property "Part Number" "114-TG2520SMN38.4000M-MCGNNM3CT-ND"
+			(at 0 0 180)
+			(unlocked yes)
+			(layer "F.Fab")
+			(hide yes)
+			(effects
+				(font
+					(size 1 1)
+					(thickness 0.15)
+				)
+			)
+		)
+		(property "TCXO-Footprints" "3225 or 2510"
+			(at 0 0 180)
+			(unlocked yes)
+			(layer "F.Fab")
+			(hide yes)
+			(effects
+				(font
+					(size 1 1)
+					(thickness 0.15)
+				)
+			)
+		)
 		(property ki_fp_filters "Oscillator*SMD*ECS*2520MV*2.5x2.0mm*")
 		(sheetname "/")
 		(sheetfile "SX1255-SXCEIVER-HAT.kicad_sch")
-		(attr smd exclude_from_bom)
+		(attr smd)
 		(fp_line
 			(start -2 1.65)
@@
 		(sheetname "/")
 		(sheetfile "SX1255-SXCEIVER-HAT.kicad_sch")
-		(attr smd)
+		(attr smd exclude_from_bom dnp)
 		(fp_line
 			(start 0.8 -0.735)
@@
 		(sheetname "/")
 		(sheetfile "SX1255-SXCEIVER-HAT.kicad_sch")
-		(attr smd)
+		(attr smd exclude_from_bom dnp)
 		(fp_line
 			(start -0.237258 -0.5225)
@@
 			(layers "F.Cu" "F.Mask" "F.Paste")
 			(roundrect_rratio 0.125)
-			(net 2 "GND")
 			(solder_mask_margin 0.102)
 		)
@@
 			(layers "F.Cu" "F.Mask" "F.Paste")
 			(roundrect_rratio 0.125)
-			(net 2 "GND")
 			(solder_mask_margin 0.102)
 		)
@@
 			(layers "F.Cu" "F.Mask" "F.Paste")
 			(roundrect_rratio 0.125)
-			(net 2 "GND")
 			(solder_mask_margin 0.102)
 		)
@@
 			(layers "F.Cu" "F.Mask" "F.Paste")
 			(roundrect_rratio 0.125)
-			(net 2 "GND")
 			(solder_mask_margin 0.102)
 		)
@@
 			(layers "F.Cu" "F.Mask" "F.Paste")
 			(roundrect_rratio 0.125)
-			(net 2 "GND")
 			(solder_mask_margin 0.102)
 		)
@@
 		(sheetname "/")
 		(sheetfile "SX1255-SXCEIVER-HAT.kicad_sch")
-		(attr smd)
+		(attr smd exclude_from_bom dnp)
 		(fp_line
 			(start 0.8 -0.735)
