File: SX1255-SXCEIVER-HAT.kicad_sch (KiCad schematic)
At the start: 90 parts, among them IC1 SX1255, J1 U.FL, J2 U.FL, J3 RPi, J4 WP, Q1 BSS84, SW1 SW_Push, U1 MCP1703Ax-330xxDB, U2 24LC256, U3 74LVC1G74DP_125, U4 TQP3M9036, Y1 TCXO 38.40MHz

Commit message: Add files via upload
Other:
- moved on the sheet: C12, C13, D1, J4, R10, R11, R12, R13, R15, R33, R5, R6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

Commit message: Add files via upload
Parts:
- C16, D2, D3, R32, R34, R35, SW1: now left out of the parts list
Changed lines of the file:
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@@
 	(title_block
 		(title "SX1255 RPi 4-5 HAT")
-		(date "2026-03-01")
+		(date "2026-03-02")
 		(rev "V1.3")
 		(company "Z32IT")
@@
 		(unit 1)
 		(exclude_from_sim yes)
-		(in_bom yes)
-		(on_board yes)
+		(in_bom no)
+		(on_board no)
 		(dnp no)
 		(property "Reference" "D2"
@@
 		(unit 1)
 		(exclude_from_sim yes)
-		(in_bom yes)
-		(on_board yes)
+		(in_bom no)
+		(on_board no)
 		(dnp no)
 		(property "Reference" "R34"
@@
 		(unit 1)
 		(exclude_from_sim yes)
-		(in_bom yes)
-		(on_board yes)
+		(in_bom no)
+		(on_board no)
 		(dnp no)
 		(property "Reference" "R35"
@@
 		(unit 1)
 		(exclude_from_sim yes)
-		(in_bom yes)
-		(on_board yes)
+		(in_bom no)
+		(on_board no)
 		(dnp no)
 		(property "Reference" "D3"
@@
 		(unit 1)
 		(exclude_from_sim yes)
-		(in_bom yes)
-		(on_board yes)
+		(in_bom no)
+		(on_board no)
 		(dnp no)
 		(property "Reference" "R32"
@@
 		(at 347.98 120.65 0)
 		(unit 1)
-		(exclude_from_sim no)
+		(exclude_from_sim yes)
 		(in_bom no)
 		(on_board yes)
@@
 		(unit 1)
 		(exclude_from_sim yes)
-		(in_bom yes)
-		(on_board yes)
+		(in_bom no)
+		(on_board no)
 		(dnp no)
 		(fields_autoplaced yes)
@@
 		(unit 1)
 		(exclude_from_sim yes)
-		(in_bom yes)
-		(on_board yes)
+		(in_bom no)
+		(on_board no)
 		(dnp no)
 		(property "Reference" "C16"

Commit message: Add files via upload
Parts:
- removed F1: 6V/0.5A, Fuse:Fuse_1206_3216Metric, symbol Device:Polyfuse_Small
- C1, C10, C11, C15, C3, C30: Manufacturer (none) -> YAGEO; Manufacturer Product Number (none) -> CC0603JRX7R6BB105; Part Number (none) -> 311-3484-1-ND
- C12, C13, C14, C4, C7, C8, C9: Manufacturer (none) -> Vishay Vitramon; Manufacturer Product Number (none) -> VJ0603Y104JXQPW1BC; Part Number (none) -> 720-1688-1-ND
- C17, C19, C28, C31: Manufacturer (none) -> KEMET; Manufacturer Product Number (none) -> C0603C101J8GACTU; Part Number (none) -> 399-15348-1-ND
- C18: Manufacturer (none) -> KEMET; Manufacturer Product Number (none) -> C0603C103K8RACTU; Part Number (none) -> 399-C0603C103K8RACTUCT-ND
- C2, C5: Manufacturer (none) -> Samsung Electro-Mechanics; Manufacturer Product Number (none) -> CL31B226MPHNNNE; Part Number (none) -> 1276-3148-1-ND
- C6: Manufacturer (none) -> KEMET; Manufacturer Product Number (none) -> C0603C100J8GACTU; Part Number (none) -> 399-14932-1-ND; now left out of the parts list
- D1: Manufacturer (none) -> Lite-On Inc.; Manufacturer Product Number (none) -> LTST-T180UWET; Part Number (none) -> 160-LTST-T180UWETCT-ND
- D2: Manufacturer (none) -> Kingbright; Manufacturer Product Number (none) -> APT1608SGD3; Part Number (none) -> 754-APT1608SGD3CT-ND; now in the parts list
- D3: Manufacturer (none) -> Lite-On Inc.; Manufacturer Product Number (none) -> LTST-S270KRKT; Part Number (none) -> 160-1479-1-ND; now in the parts list
- D4, D5: Manufacturer (none) -> Lite-On Inc.; Manufacturer Product Number (none) -> LTST-C190KSKT; Part Number (none) -> 160-1437-1-ND
- D6, D7: Manufacturer (none) -> Kingbright; Manufacturer Product Number (none) -> APT1608SGD3; Part Number (none) -> 754-APT1608SGD3CT-ND
- FL1, FL2: Manufacturer (none) -> Mini-Circuits; Manufacturer Product Number (none) -> LFCN-490+; Part Number (none) -> 3157-LFCN-490+CT-ND
- IC1: Height 0.8 -> (none); MPN SX1255IWLTRT -> (none); Manufacturer (none) -> Semtech Corporation; Manufacturer Product Number (none) -> SX1255IWLTRT; PN 947-SX1255IWLTRT -> (none); Part Number (none) -> SX1255IWLTRTCT-ND
- J1, J2: Manufacturer (none) -> TE Connectivity Linx; Manufacturer Product Number (none) -> CONMHF1-SMD-G-T; PROD_ID CONN-09193 -> (none); Part Number (none) -> 343-CONMHF1-SMD-G-TCT-ND
- J3: MPN - -> (none); PN - -> (none)
- J4: now left out of the parts list
- L1: Manufacturer (none) -> Murata Electronics; Manufacturer Product Number (none) -> BLM18HG601SN1D; Part Number (none) -> 490-1033-1-ND
- L2: Manufacturer (none) -> Johanson Technology Inc.; Manufacturer Product Number (none) -> LRC0603CJ82NGV001T; Part Number (none) -> 712-LRC0603CJ82NGV001TCT-ND
- L3: Manufacturer (none) -> Johanson Technology Inc.; Manufacturer Product Number (none) -> LRC0603CJ39NGV001T; Part Number (none) -> 712-LRC0603CJ39NGV001TCT-ND
- L4: footprint Capacitor_SMD:C_0603_1608Metric -> Inductor_SMD:L_0603_1608Metric;  Part Number (none) -> 712-LRC0603CJ68NGV001TCT-ND; Manufacturer (none) -> Johanson Technology Inc.; Manufacturer Product Number (none) -> LRC0603CJ68NGV001T
- Q1: Manufacturer (none) -> MDD; Manufacturer Product Number (none) -> BSS84; Part Number (none) -> 3372-BSS84TR-ND
- R1: Manufacturer (none) -> Vishay Dale; Manufacturer Product Number (none) -> CRCW060310K0FKEA; Part Number (none) -> 541-10.0KHCT-ND; now left out of the parts list
- R10: Manufacturer (none) -> Vishay Dale; Manufacturer Product Number (none) -> CRCW06031K00FKEA; Part Number (none) -> 541-1.00KHCT-ND
- R11, R13, R26, R27: Manufacturer (none) -> Vishay Dale; Manufacturer Product Number (none) -> CRCW06031M00FKEA; Part Number (none) -> 541-1.00MHCT-ND
- R12, R17, R18, R19, R21, R23, R24, R30, R5, R6, R8: Manufacturer (none) -> Vishay Dale; Manufacturer Product Number (none) -> CRCW0603330RFKEA; Part Number (none) -> 541-330HCT-ND
- R14, R16, R20, R22, R28: Manufacturer (none) -> Vishay Dale; Manufacturer Product Number (none) -> CRCW060333R0FKEA; Part Number (none) -> 541-33.0HCT-ND
- R15, R38, R39, R9: Manufacturer (none) -> Vishay Dale; Manufacturer Product Number (none) -> CRCW06033K30FKEA; Part Number (none) -> 541-3.30KHCT-ND
- R2, R7: Manufacturer (none) -> Vishay Dale; Manufacturer Product Number (none) -> CRCW06030000Z0EA; Part Number (none) -> 541-0.0GCT-ND
- R25: Manufacturer (none) -> Vishay Dale; Manufacturer Product Number (none) -> CRCW060310K0FKEA; Part Number (none) -> 541-10.0KHCT-ND
- R3, R31, R4: Manufacturer (none) -> Vishay Dale; Manufacturer Product Number (none) -> CRCW06031R00FKEA; Part Number (none) -> 541-1.00HHCT-ND
- R33, R36, R37: Manufacturer (none) -> Vishay Dale; Manufacturer Product Number (none) -> CRCW06031K50JNEA; Part Number (none) -> 541-1.5KGCT-ND
- R34: Manufacturer (none) -> Vishay Dale; Manufacturer Product Number (none) -> CRCW06031K00FKEA; Part Number (none) -> 541-1.00KHCT-ND; now in the parts list
- R35: Manufacturer (none) -> Vishay Dale; Manufacturer Product Number (none) -> CRCW0603330RFKEA; Part Number (none) -> 541-330HCT-ND; now in the parts list
- U1: Manufacturer (none) -> Microchip Technology; Manufacturer Product Number (none) -> MCP1703T-3302E/DB; Part Number (none) -> MCP1703T-3302E/DBCT-ND
- U2: Manufacturer (none) -> Microchip Technology; Manufacturer Product Number (none) -> 24LC256-I/SN; Part Number (none) -> 24LC256-I/SN-ND
- U3: Availability In Stock -> (none); Check_prices https://www.snapeda.com/parts/74LVC1G74DP,125/NXP+Semicondu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 -> (none); DESCRIPTION 74LVC1G74 - Single D-type flip-flop with set and reset; pos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 -> (none); Description_1 Flip Flop 1 Element D-Type 1 Bit Positive Edge 8-TSSOP, 8-M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 -> (none); HEIGHT 1.1mm -> (none); MANUFACTURER_NAME Nexperia -> (none); MANUFACTURER_PART_NUMBER 74LVC1G74DP,125 -> (none); MF NXP USA Inc. -> (none); MOUSER_PART_NUMBER 771-LVC1GDP125 -> (none); MOUSER_PRICE-STOCK https://www.mouser.co.uk/ProductDetail/Nexperia/74LVC1G74DP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 -> (none); MP 74LVC1G74DP,125 -> (none); Manufacturer (none) -> Nexperia USA Inc.; Manufacturer Product Number (none) -> 74LVC1G74DP,125; Package TSSOP8-8 Nexperia USA Inc. -> (none); Part Number (none) -> 1727-5983-1-ND; Price None -> (none); SnapEDA_Link https://www.snapeda.com/parts/74LVC1G74DP,125/NXP+Semicondu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 -> (none)
- U4: Availability In Stock -> (none); Check_prices https://www.snapeda.com/parts/TQP3M9036/Qorvo/view-part/?re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 -> (none); Description_1 RF Amp Chip Single GP 2GHz 5.25V 8-Pin DFN EP T/R -> (none); MANUFACTURER Qorvo -> (none); MAXIMUM_PACKAGE_HEIGHT 0.95mm -> (none); MF Qorvo -> (none); MP TQP3M9036 -> (none); Manufacturer (none) -> Qorvo; Manufacturer Product Number (none) -> TQP3M9036; PARTREV N/A -> (none); Package DFN-8 Qorvo -> (none); Part Number (none) -> 2312-TQP3M9036CT-ND; Price None -> (none); Purchase-URL https://www.snapeda.com/api/url_track_click_mouser/?unipart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 -> (none); STANDARD IPC-7351B -> (none); SnapEDA_Link https://www.snapeda.com/parts/TQP3M9036/Qorvo/view-part/?re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 -> (none)
- Y1: value TCXO 38.40MHz -> 38.4MHz; footprint Crystal:Crystal_SMD_3225-4Pin_3.2x2.5mm -> Oscillator:Oscillator_SMD_ECS_2520MV-xxx-xx-4Pin_2.5x2.0mm; Manufacturer (none) -> EPSON; Manufacturer Product Number (none) -> TG2520SMN 38.4000M-MCGNNM3; Part Number (none) -> 114-TG2520SMN38.4000M-MCGNNM3CT-ND
Connections:
- net +5VP: now also C1.1, L1.1

Commit message: Add files via upload
Parts:
- removed C16: 10n, Capacitor_SMD:C_0603_1608Metric, symbol Device:C_Small
- removed R32: 330R, Resistor_SMD:R_0603_1608Metric, symbol Device:R_Small
- removed SW1: SW_Push, Button_Switch_SMD:SW_Push_1P1T_NO_E-Switch_TL3301NxxxxxG, symbol Switch:SW_Push
- added JP1: With/Without U3, Jumper:SolderJumper-2_P1.3mm_Open_RoundedPad1.0x1.5mm, symbol Jumper:SolderJumper_2_Open
- L1: footprint Inductor_SMD:L_0603_1608Metric -> Inductor_SMD:L_0805_2012Metric
- Y1: value 38.4MHz -> 38.4MHZ; footprint Oscillator:Oscillator_SMD_ECS_2520MV-xxx-xx-4Pin_2.5x2.0mm -> Crystal:Crystal_SMD_3225-4Pin_3.2x2.5mm; Manufacturer EPSON -> (none); Manufacturer Product Number TG2520SMN 38.4000M-MCGNNM3 -> (none); Model (none) -> KDS-DSB321SDN or other brands; Part Number 114-TG2520SMN38.4000M-MCGNNM3CT-ND -> (none); now left out of the parts list
Connections:
- net SX_VBAT3: now also JP1.2 (B)
- net at C15.1, Q1.2 (S), R31.1: now also JP1.1 (A)
Other:
- note added: "JP1, Closed, Without Q1 and R30, U3 and components around it."
- note added: "JP1, Open, Standard schematic"

Commit message: Add files via upload
Parts:
- L1: Manufacturer Product Number BLM18HG601SN1D -> BLM21BD601SN1D; Part Number 490-1033-1-ND -> 490-1046-1-ND
- Y1: value 38.4MHZ -> 38.4MHz; Manufacturer (none) -> EPSON; Manufacturer Product Number (none) -> TG2520SMN 38.4000M-MCGNNM3; Model KDS-DSB321SDN or other brands -> (none); Part Number (none) -> 114-TG2520SMN38.4000M-MCGNNM3CT-ND; TCXO-Footprints (none) -> 3225 or 2510; now in the parts list
Changed lines of the file:
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@@
 		(title "SX1255 RPi 4-5 HAT")
 		(date "2026-03-15")
-		(rev "V1.3.2")
+		(rev "V1.3.2 FINAL")
 		(company "Z32IT")
 		(comment 1 "Modified SXceiver")
 	)
-	(text "JP1, Open, Standard schematic"
+	(text "JP1, Closed, Without Q1 and R30, U3 and components around it."
 		(exclude_from_sim no)
-		(at 134.62 98.806 0)
+		(at 134.366 104.394 0)
 		(effects
 			(font
@@
 		)
 	)
-	(text "TX-LED"
+	(text "JP1, Open, Standard schematic"
 		(exclude_from_sim no)
-		(at 168.656 236.728 0)
+		(at 133.096 101.092 0)
 		(effects
 			(font
@@
 		)
 	)
-	(text "JP1, Closed, Without Q1 and R30, U3 and components around it."
+	(text "TX-LED"
 		(exclude_from_sim no)
-		(at 135.89 102.108 0)
+		(at 168.656 236.728 0)
 		(effects
 			(font
@@
 	(wire
 		(pts
-			(xy 177.8 86.36) (xy 187.96 86.36)
-		)
-		(stroke
-			(width 0)
-			(type default)
-		)
-	)
-	(wire
-		(pts
 			(xy 250.19 68.58) (xy 262.89 68.58)
 		)
@@
 	(wire
 		(pts
-			(xy 165.1 86.36) (xy 165.1 93.98)
-		)
-		(stroke
-			(width 0)
-			(type default)
-		)
-	)
-	(wire
-		(pts
 			(xy 59.69 110.49) (xy 57.15 110.49)
 		)
@@
 	(wire
 		(pts
-			(xy 170.18 86.36) (xy 165.1 86.36)
+			(xy 219.71 227.33) (xy 224.79 227.33)
 		)
 		(stroke
@@
 	(wire
 		(pts
-			(xy 219.71 227.33) (xy 224.79 227.33)
+			(xy 173.99 227.33) (xy 177.8 227.33)
 		)
 		(stroke
@@
 	(wire
 		(pts
-			(xy 173.99 227.33) (xy 177.8 227.33)
+			(xy 170.18 86.36) (xy 165.1 86.36)
 		)
 		(stroke
@@
 	(wire
 		(pts
+			(xy 165.1 86.36) (xy 165.1 93.98)
+		)
+		(stroke
+			(width 0)
+			(type default)
+		)
+	)
+	(wire
+		(pts
 			(xy 172.72 68.58) (xy 182.88 68.58)
 		)
@@
 	(wire
 		(pts
-			(xy 187.96 86.36) (xy 187.96 93.98)
-		)
-		(stroke
-			(width 0)
-			(type default)
-		)
-	)
-	(wire
-		(pts
 			(xy 187.96 121.92) (xy 190.5 121.92)
 		)
@@
 	(wire
 		(pts
+			(xy 187.96 86.36) (xy 187.96 93.98)
+		)
+		(stroke
+			(width 0)
+			(type default)
+		)
+	)
+	(wire
+		(pts
 			(xy 354.33 167.64) (xy 356.87 167.64)
 		)
@@
 	(wire
 		(pts
+			(xy 177.8 86.36) (xy 187.96 86.36)
+		)
+		(stroke
+			(width 0)
+			(type default)
+		)
+	)
+	(wire
+		(pts
 			(xy 236.22 137.16) (xy 243.84 137.16)
 		)
@@
 	)
 	(symbol
-		(lib_id "Oscillator:ECS-2520MV-xxx-xx")
-		(at 68.58 129.54 0)
-		(unit 1)
-		(exclude_from_sim no)
-		(in_bom no)
-		(on_board yes)
-		(dnp no)
-		(property "Reference" "Y1"
-			(at 64.262 122.428 0)
-			(effects
-				(font
-					(size 1.27 1.27)
-				)
-			)
-		)
-		(property "Value" "38.4MHZ"
-			(at 68.58 129.286 0)
-			(effects
-				(font
-					(size 1.27 1.27)
-				)
-			)
-		)
-		(property "Footprint" "Crystal:Crystal_SMD_3225-4Pin_3.2x2.5mm"
-			(at 80.01 138.43 0)
-			(effects
-				(font
-					(size 1.27 1.27)
-				)
-				(hide yes)
-			)
-		)
-		(property "Datasheet" "~"
-			(at 64.135 126.365 0)
-			(effects
-				(font
-					(size 1.27 1.27)
-				)
-				(hide yes)
-			)
-		)
-		(property "Description" "Clipped SW 0.5~1ppm"
-			(at 77.47 122.428 0)
-			(effects
-				(font
-					(size 1 1)
-				)
-			)
-		)
-		(property "Model" "KDS-DSB321SDN or other brands"
-			(at 85.598 119.888 0)
-			(effects
-				(font
-					(size 1.27 1.27)
-				)
-			)
-		)
-		(pin "1"
-		)
-		(pin "3"
-		)
-		(pin "2"
-		)
-		(pin "4"
-		)
-		(instances
-			(project "SX1255-SXCEIVER-HAT"
-				(path "/5946dd4e-fab1-4214-b6c7-4fabd0e98d1f"
-					(reference "Y1")
-					(unit 1)
-				)
-			)
-		)
-	)
-	(symbol
 		(lib_id "Device:R_Small")
 		(at 351.79 167.64 270)
@@
 	)
 	(symbol
+		(lib_name "ECS-2520MV-xxx-xx_1")
+		(lib_id "Oscillator:ECS-2520MV-xxx-xx")
+		(at 68.58 129.54 0)
+		(unit 1)
+		(exclude_from_sim no)
+		(in_bom yes)
+		(on_board yes)
+		(dnp no)
+		(property "Reference" "Y1"
+			(at 64.77 121.666 0)
+			(effects
+				(font
+					(size 1.27 1.27)
+				)
+			)
+		)
+		(property "Value" "38.4MHz"
+			(at 68.834 128.778 0)
+			(effects
+				(font
+					(size 1.27 1.27)
+				)
+			)
+		)
+		(property "Footprint" "Crystal:Crystal_SMD_3225-4Pin_3.2x2.5mm"
+			(at 80.01 138.43 0)
+			(effects
+				(font
+					(size 1.27 1.27)
+				)
+				(hide yes)
+			)
+		)
+		(property "Datasheet" "~"
+			(at 64.135 126.365 0)
+			(effects
+				(font
+					(size 1.27 1.27)
+				)
+				(hide yes)
+			)
+		)
+		(property "Description" "Clipped SW/0.5~1ppm"
+			(at 80.264 122.428 0)
+			(effects
+				(font
+					(size 1.27 1.27)
+				)
+			)
+		)
+		(property "Manufacturer" "EPSON "
+			(at 68.58 129.54 0)
+			(effects
+				(font
+					(size 1.27 1.27)
+				)
+				(hide yes)
+			)
+		)
+		(property "Manufacturer Product Number" "TG2520SMN 38.4000M-MCGNNM3"
+			(at 68.58 129.54 0)
+			(effects
+				(font
+					(size 1.27 1.27)
+				)
+				(hide yes)
+			)
+		)
+		(property "Part Number" "114-TG2520SMN38.4000M-MCGNNM3CT-ND"
+			(at 68.58 129.54 0)
+			(effects
+				(font
+					(size 1.27 1.27)
+				)
+				(hide yes)
+			)
+		)
+		(property "TCXO-Footprints" "3225 or 2510"
+			(at 68.58 129.54 0)
+			(effects
+				(font
+					(size 1.27 1.27)
+				)
+				(hide yes)
+			)
+		)
+		(pin "2"
+		)
+		(pin "3"
+		)
+		(pin "4"
+		)
+		(pin "1"
+		)
+		(instances
+			(project ""
+				(path "/5946dd4e-fab1-4214-b6c7-4fabd0e98d1f"
+					(reference "Y1")
+					(unit 1)
+				)
+			)
+		)
+	)
+	(symbol
 		(lib_id "power:GND")
 		(at 238.76 158.75 90)
@@
 			)
 		)
-		(property "Description" "Inductor with ferrite core, small symbol"
+		(property "Description" "FERRITE BEAD 600 OHM 0805 1LN"
 			(at 60.96 177.8 0)
 			(effects
@@
 			)
 		)
-		(property "Manufacturer Product Number" "BLM18HG601SN1D"
+		(property "Manufacturer Product Number" "BLM21BD601SN1D"
 			(at 60.96 177.8 90)
 			(effects
@@
 			)
 		)
-		(property "Part Number" "490-1033-1-ND"
+		(property "Part Number" "490-1046-1-ND"
 			(at 60.96 177.8 90)
 			(effects
@@
 		)
 		(instances
-			(project ""
+			(project "SX1255-SXCEIVER-HAT"
 				(path "/5946dd4e-fab1-4214-b6c7-4fabd0e98d1f"
 					(reference "L1")
