File: SX1255-SXCEIVER-HAT with BPF/SX1255-SXCEIVER-HAT with BPF.kicad_pcb (KiCad board)
At the start: 2 copper layers, 65 x 56.2 mm, 84 parts, among them IC1 SX1255, J1 TX_SMA, J2 RX_SMA, J3 RPi, J4 WP, Q1 BSS84, U1 MCP1703Ax-330xxDB, U2 24LC256, U3 74LVC1G74DP_125, U4 TQP3M9036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

Commit message: Add files via upload
Parts:
- removed F1: 6V/0.5A, Fuse:Fuse_1206_3216Metric
- added D2: Green, LED_SMD:LED_0603_1608Metric_Pad1.05x0.95mm_HandSolder, F.Cu at (158.0, 91.3)
- added D3: Red, LED_SMD:LED_0603_1608Metric_Pad1.05x0.95mm_HandSolder, F.Cu at (159.8, 91.3)
- added R34: 1K, Resistor_SMD:R_0603_1608Metric, F.Cu at (158.0, 87.8)
- added R35: 330R, Resistor_SMD:R_0603_1608Metric, F.Cu at (159.8, 87.8)
- Y1: value TCXO 38.40MHz -> 38.4MHz; footprint Crystal:Crystal_SMD_3225-4Pin_3.2x2.5mm -> Oscillator:Oscillator_SMD_ECS_2520MV-xxx-xx-4Pin_2.5x2.0mm
- moved C1 7.28 mm to (110.0, 78.8), turned to 0 degrees
- moved L1 2.36 mm to (106.8, 79.5)
- moved R2 0.25 mm to (147.5, 92.0)
- moved Y1 0.22 mm to (146.4, 96.0), turned to -90 degrees
Connections:
- C1 pad 1: Net-(C1-Pad1) -> +5VP
- L1 pad 1: Net-(C1-Pad1) -> +5VP
Routing:
- net /H_GPIO12: track 0.00 -> 25.9 mm, vias 0 -> 2
- net /H_GPIO13: track 0.00 -> 20.6 mm, vias 0 -> 2
- net Net-(C1-Pad1): track 3.87 -> 0.00 mm
- net +5VP: track 10.4 -> 13.2 mm
- net Net-(D3-A): track 0.00 -> 1.80 mm
- net Net-(D2-A): track 0.00 -> 1.80 mm
- net +5V: track 95.7 -> 97.0 mm
- net +3V3: track 101.0 -> 102.0 mm
- net GND: vias 37 -> 36
Other:
- board text added: "DIO0"
- board text added: "DIO1"
- board text added: "DIO3"
- board text added: "GPIO12"
- board text added: "GPIO13"
- board text added: "V1.4.1"
- board text removed: "V1.4(BPF)"

Commit message: Add files via upload
Other:
- board text added: "PA"
- board text added: "POW"
Changed lines of the file:
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@@
 		(layer "Edge.Cuts")
+	)
+	(gr_text "PA"
+		(at 116.5 86.25 0)
+		(layer "F.SilkS")
+		(effects
+			(font
+				(size 1 1)
+				(thickness 0.25)
+				(bold yes)
+			)
+			(justify left bottom)
+		)
 	)
 	(gr_text "GPIO12"
@@
 		(layer "F.SilkS")
 		(effects
+			(font
+				(size 1 1)
+				(thickness 0.25)
+				(bold yes)
+			)
+			(justify left bottom)
+		)
+	)
+	(gr_text "POW"
+		(at 119.5 91.25 0)
+		(layer "F.SilkS")
+		(effects
