File: SX1255-SXCEIVER-HAT with BPF/SX1255-SXCEIVER-HAT with BPF.kicad_pcb (KiCad board)
At the start: 2 copper layers, 65 x 56.2 mm, 87 parts, among them IC1 SX1255, J1 TX_SMA, J2 RX_SMA, J3 RPi, J4 WP, Q1 BSS84, U1 MCP1703Ax-330xxDB, U2 24LC256, U3 74LVC1G74DP_125, U4 TQP3M9036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

Commit message: Add files via upload
Parts:
- L1: footprint Inductor_SMD:L_0603_1608Metric -> Inductor_SMD:L_0805_2012Metric
- Y1: value 38.4MHz -> 38.4MHZ; footprint Oscillator:Oscillator_SMD_ECS_2520MV-xxx-xx-4Pin_2.5x2.0mm -> Crystal:Crystal_SMD_3225-4Pin_3.2x2.5mm
- moved L4 2.70 mm to (144.2, 113.2)
- moved C30 2.50 mm to (143.5, 118.2)
- moved C31 2.30 mm to (143.5, 116.8)
- moved REF** 2.12 mm to (127.2, 120.0)
- moved R26 1.25 mm to (114.5, 112.8)
- moved C1 0.50 mm to (110.0, 78.2)
- moved X1 0.50 mm to (120.1, 112.0)
- moved R2 0.35 mm to (147.8, 91.8)
- moved L1 0.25 mm to (106.8, 79.2)
- moved Y1 0.22 mm to (146.6, 95.8), turned to 180 degrees
Routing:
- net /RF-out: track 5.97 -> 3.52 mm
- net +3V3: track 102.0 -> 101.2 mm
- net +5VP: track 13.2 -> 12.7 mm
- net Net-(X1-OUT): track 3.04 -> 3.54 mm
- net GND: vias 36 -> 271
Other:
- board text added: "V1.4.2"
- board text added: "m/SXceiver"
- board text removed: "V1.4.1"

Commit message: Add files via upload
Parts:
- added JP1: With/Without U3, Jumper:SolderJumper-2_P1.3mm_Open_RoundedPad1.0x1.5mm, F.Cu at (150.5, 99.5)
Routing:
- net /SX_VBAT3: track 17.1 -> 22.3 mm
- net Net-(JP1-A): track 3.76 -> 8.64 mm
- net GND: vias 271 -> 273

Commit message: Add files via upload
Other:
- board text added: "Duplex 7.6 ~ 10MHz"
Changed lines of the file:
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@@
+		)
+	)
+	(gr_text "Duplex 7.6 ~ 10MHz"
+		(at 146.75 121.25 0)
+		(layer "F.SilkS")
+		(effects
+			(font
+				(size 0.7 0.7)
+				(thickness 0.175)
+				(bold yes)
+			)
+			(justify left bottom)
 		)
 	)

Commit message: Add files via upload
Other:
- board text added: "V1.4.3"
- board text removed: "V1.4.2"
Changed lines of the file:
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@@
 	(title_block
 		(title "SX1255-SXceiver-HAT with BPF")
-		(date "2026-03-08")
-		(rev "V1.4.2")
+		(date "2026-03-15")
+		(rev "V1.4.3 Final")
 		(company "Z32IT")
 		(comment 1 "Modified SXceiver")
@@
 		(sheetname "/")
 		(sheetfile "SX1255-SXCEIVER-HAT with BPF.kicad_sch")
-		(attr smd)
+		(attr smd exclude_from_bom dnp)
 		(fp_line
 			(start -0.237258 -0.5225)
@@
 		(sheetname "/")
 		(sheetfile "SX1255-SXCEIVER-HAT with BPF.kicad_sch")
-		(attr smd)
+		(attr smd exclude_from_bom dnp)
 		(fp_line
 			(start 0.8 -0.735)
@@
 		(sheetname "/")
 		(sheetfile "SX1255-SXCEIVER-HAT with BPF.kicad_sch")
-		(attr smd)
+		(attr smd exclude_from_bom dnp)
 		(fp_line
 			(start 0.8 -0.735)
@@
 		(sheetname "/")
 		(sheetfile "SX1255-SXCEIVER-HAT with BPF.kicad_sch")
-		(attr smd)
+		(attr smd exclude_from_bom dnp)
 		(fp_line
 			(start -0.237258 -0.5225)
@@
 		)
 	)
-	(gr_text "V1.4.2"
+	(gr_text "V1.4.3"
 		(at 131.75 121.75 0)
 		(layer "F.SilkS")
