File: SX1255-SXCEIVER-HAT_microspot/SX1255-SXCEIVER-HAT_microspot.kicad_pcb (KiCad board)
At the start: 2 copper layers, 65 x 56.2 mm, 84 parts, among them IC1 SX1255, J3 RPi, J4 WP, Q1 BSS84, U1 MCP1703Ax-330xxDB, U2 24LC256, U3 74LVC1G74DP_125, X1 TA0655A, X2 TA1761A, Y1 38.4MHZ

Commit message: Add files via upload
Parts:
- removed E2: RX-CHP, ANT-868-CHP-T:XDCR_ANT-868-CHP-T
- added E1: TX-CHP, ANT-868-CHP-T:CrossAir_CA-S01, F.Cu at (110.0, 116.2)
- E1: footprint ANT-868-CHP-T:XDCR_ANT-868-CHP-T -> ANT-868-CHP-T:CrossAir_CA-S01
Routing:
- net GND: vias 32 -> 424

Commit message: Add files via upload
Parts:
- added JP1: With/Without U3, Jumper:SolderJumper-2_P1.3mm_Open_RoundedPad1.0x1.5mm, F.Cu at (150.5, 99.5)
- E1: footprint ANT-868-CHP-T:CrossAir_CA-S01 -> ANT-868-CHP-T:XDCR_ANT-868-CHP-T
- E2: renamed from E1; footprint ANT-868-CHP-T:CrossAir_CA-S01 -> ANT-868-CHP-T:XDCR_ANT-868-CHP-T
Routing:
- net Net-(JP1-A): track 3.76 -> 8.85 mm
- net /SX_VBAT3: track 17.1 -> 22.2 mm
- net GND: vias 424 -> 426
Other:
- board text added: "Duplex 7.6 ~ 10MHz"
