File: SX1255-SXCEIVER-HAT_microspot/SX1255-SXCEIVER-HAT_microspot.kicad_sch (KiCad schematic)
At the start: 86 parts, among them IC1 SX1255, J3 RPi, J4 WP, Q1 BSS84, SW1 SW_Push, U1 MCP1703Ax-330xxDB, U2 24LC256, U3 74LVC1G74DP_125, X1 TA0655A, X2 TA1761A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

Commit message: Add files via upload
Parts:
- Y1: Model KDS-DSA321SDN -> KDS-DSB321SDN
Changed lines of the file:
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@@
 			)
 		)
-		(property "Model" "KDS-DSA321SDN"
+		(property "Model" "KDS-DSB321SDN"
 			(at 77.47 119.634 0)
 			(effects

Commit message: Add files via upload
Parts:
- added JP1: With/Without U3, Jumper:SolderJumper-2_P1.3mm_Open_RoundedPad1.0x1.5mm, symbol Jumper:SolderJumper_2_Open
Connections:
- net SX_VBAT3: now also JP1.2 (B)
- net at C15.1, Q1.2 (S), R31.1: now also JP1.1 (A)
Other:
- note added: "JP1, Closed, Without Q1-R30, U3 and components around it."
- note added: "JP1, Open, Standard schematic"
- moved on the sheet: C15, C19, E1, E2, L2, L3, L5, L6, R26, R27, R31, X1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

Commit message: Add files via upload
Parts:
- removed C16: 10n, Capacitor_SMD:C_0603_1608Metric, symbol Device:C_Small
- removed R32: 330R, Resistor_SMD:R_0603_1608Metric, symbol Device:R_Small
- removed SW1: SW_Push, Button_Switch_SMD:SW_Push_1P1T_NO_E-Switch_TL3301NxxxxxG, symbol Switch:SW_Push
